File: kicad/nametag.kicad_sch (KiCad schematic)
At the start: 85 parts, among them J2 FPC24 0.5mm, J3 Prog Header, Q1 Si1308EDL, Q2 AO3401A, Q3 AO3401A, SW2 SW_Push, U2 nRF52832-QFxx, Y2 Crystal_GND24

Commit message: First routing
Did the routing for everything and made it somewhat useable.
Have to sleep again for a night to see if I want to do it like this.
Parts:
- removed D11, D15, D16, D17, D18, D19, D21: LED, g-LED_SMD:LTST-C230, symbol Device:LED
- removed R15, R19, R20, R21, R22, R23, R25: R, Resistor_SMD:R_0603_1608Metric, symbol Device:R
- L1: value L -> 68uH; footprint (none) -> Inductor_SMD:L_1210_3225Metric
Connections:
- net LED_3 is gone; now on net LED_8: D6.1 (K)
- net BUSY: now also U2.17 (P0.14)
- net CS: now also U2.20 (P0.17)
- net DATA/CLOCK: now also U2.19 (P0.16)
- net ENABLE: now also U2.16 (P0.13)
- net LED: now also U2.14 (P0.11); no longer U2.19 (P0.16)
- net LED-POWER: now also U2.15 (P0.12)
- net LED_1: now also U2.9 (P0.07)
- net LED_10: now also U2.10 (P0.08)
- net LED_11: now also U2.12 (NFC2/P0.10)
- net LED_17: now also U2.2 (P0.00/XL1)
- net LED_2: now also U2.11 (NFC1/P0.09)
- net LED_4: now also U2.4 (P0.02/AIN0)
- net LED_5: now also U2.8 (P0.06)
- net LED_6: now also U2.3 (P0.01/XL2)
- net LED_7: now also U2.5 (P0.03/AIN1)
- net LED_8: now also U2.7 (P0.05/AIN3)
- net LED_9: now also U2.28 (P0.23)
- net SCK: now also U2.21 (P0.18/SWO)
- net SDI: now also U2.22 (P0.19)
- net eP_RESET: now also U2.18 (P0.15)
- net at C1.1, C2.1, J2.15 (Pin_15)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: now also L1.2; no longer L1.1
- net at C11.2, D3.2 (A), Q1.3 (D): now also L1.1; no longer L1.2
- net SWO: no longer names the net of J3.6 (SWO)
- no-connect marks 4 -> 15
Other:
- note added: "Blinky Parade"
- note added: "Debug"
- note added: "MCU"
- note added: "e-Paper Display"
- moved on the sheet: AE2, C16, C26, D20, D5, D9, H1, L1, L5, Q3, R13, R24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
