File: kicad/nametag.kicad_sch (KiCad schematic)
At the start: 71 parts, among them J2 FPC24 0.5mm, J3 Prog Header, Q1 Si1308EDL, Q2 AO3401A, Q3 AO3401A, SW2 SW_Push, U2 nRF52832-QFxx, Y2 Crystal_GND24

Commit message: old working dir
Parts:
- Y2: value Crystal_GND24 -> 32Mhz
Changed lines of the file:
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@@
 		(effects
 			(font
-				(size 1.27 1.27)
+				(size 0.8 0.8)
 			)
 			(justify left bottom)
@@
 		(effects
 			(font
-				(size 1.27 1.27)
+				(size 0.8 0.8)
 			)
 			(justify left bottom)
@@
 			)
 		)
-		(property "Value" "Crystal_GND24"
+		(property "Value" "32Mhz"
 			(at 195.58 97.79 90)
 			(effects
